Commit message: urdf finished

File: src/universal_robot/ur_description/urdf/ur10_joint_limited_robot_mm.urdf (robot description, URDF)
Before this commit: robot ur10_mm, 12 links, 11 joints
Links:
- added link agv_link_base
- added link agv_link_mid_1
- added link agv_link_mid_2
Joints:
- added joint world_agv_joint_x: type prismatic, parent agv_link_base, child agv_link_mid_1, origin xyz=0.0 0.0 0.0 rpy=0.0 0.0 0.0, axis 1 0 0, limit lower=-10 upper=10 effort=999.0 velocity=1.0
- added joint world_agv_joint_y: type prismatic, parent agv_link_mid_1, child agv_link_mid_2, origin xyz=0.0 0.0 0.0 rpy=0.0 0.0 0.0, axis 0 1 0, limit lower=-10 upper=10 effort=10.0 velocity=1.0
- added joint world_agv_joint_z: type continuous, parent agv_link_mid_2, child agv_link, origin xyz=0.0 0.0 0.0 rpy=0.0 0.0 0.0, axis 0 0 1
- joint world_joint: child agv_link -> agv_link_base

Commit message: edit urdf

File: src/universal_robot/ur_description/urdf/ur10_joint_limited_robot_mm.urdf (robot description, URDF)
Before this commit: robot ur10_mm, 15 links, 14 joints
Joints:
- joint world_agv_joint_x: limit lower=-10 upper=10 effort=999.0 velocity=1.0 -> lower=-5 upper=5 effort=100.0 velocity=1.0
- joint world_agv_joint_y: limit lower=-10 upper=10 effort=10.0 velocity=1.0 -> lower=-5 upper=5 effort=100.0 velocity=1.0
